File: keyboard_pcb.kicad_sch (KiCad schematic)
At the start: 168 parts, among them J1 USB_C_Receptacle_USB2.0_14P, SW1 SW_Push, SW2 SW_Push, U1 NCP1117-3.3_SOT223, U2 W25Q128JVS, U3 RP2040, Y1 ABM8-272-T3

Commit message: JLPCB order placed today
Parts:
- C14: value 100nF -> 100n
Changed lines of the file:
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@@
 		(dnp no)
 		(property "Reference" "C14"
-			(at 179.324 283.21 0)
+			(at 176.53 282.956 0)
 			(effects
 				(font
@@
 			)
 		)
-		(property "Value" "100nF"
-			(at 179.324 285.75 0)
+		(property "Value" "100n"
+			(at 176.022 285.75 0)
 			(effects
 				(font
