File: keyboard_pcb.kicad_pcb (KiCad board)
At the start: 2 copper layers, 168 parts, among them J1 USB_C_Receptacle_USB2.0_14P, SW1 SW_Push, SW2 SW_Push, U1 NCP1117-3.3_SOT223, U2 W25Q128JVS, U3 RP2040, Y1 ABM8-272-T3

Commit message: updates, edge cuts
Parts:
- moved C11 67.9 mm to (349.5, 111.5)
- moved MX27 67.9 mm to (276.3, 115.9)
- moved MX57 67.9 mm to (59.6, 173.1)
- moved MX58 67.9 mm to (81.0, 173.1)
- moved MX59 67.9 mm to (102.4, 173.1)
- moved MX62 67.9 mm to (269.1, 173.1)
- moved MX63 67.9 mm to (292.9, 173.1)
- moved MX64 67.9 mm to (314.4, 173.1)
- moved MX65 67.9 mm to (333.4, 173.1)
- moved MX66 67.9 mm to (352.5, 173.1)
- moved R8 67.9 mm to (339.9, 132.7)
- moved C1 67.9 mm to (334.9, 89.1)
- moved C10 67.9 mm to (349.5, 112.6)
- moved C12 67.9 mm to (346.5, 115.8)
- moved C13 67.9 mm to (347.9, 114.4)
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Other:
- board outline added: 325.4 x 96.8 mm

Commit message: cleaned up w/ .gitignore
Routing:
- net Net-(U3-USB_DM): track 37.1 -> 39.8 mm
- net GND: track 155.9 -> 156.7 mm
Other:
- board size 325.4 x 96.8 mm -> 325.4 x 97.6 mm
Changed lines of the file:
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@@
 		(fp_arc
 			(start 9.03125 8.000001)
-			(mid 8.677729 7.853537)
+			(mid 8.677693 7.853543)
 			(end 8.53125 7.500001)
 			(stroke
@@
 		(fp_arc
 			(start 14.780039 -5.999999)
-			(mid 15.133567 -5.853539)
+			(mid 15.133602 -5.853545)
 			(end 15.280039 -5.499999)
 			(stroke
@@
 		(fp_arc
 			(start 15.28125 7.500001)
-			(mid 15.134806 7.853571)
+			(mid 15.1348 7.853536)
 			(end 14.78125 8.000001)
 			(stroke
@@
 		(fp_arc
 			(start 9.03125 8.000001)
-			(mid 8.677729 7.853537)
+			(mid 8.677693 7.853543)
 			(end 8.53125 7.500001)
 			(stroke
@@
 		(fp_arc
 			(start 14.780039 -5.999999)
-			(mid 15.133567 -5.853539)
+			(mid 15.133602 -5.853545)
 			(end 15.280039 -5.499999)
 			(stroke
@@
 		(fp_arc
 			(start 15.28125 7.500001)
-			(mid 15.134806 7.853571)
+			(mid 15.1348 7.853536)
 			(end 14.78125 8.000001)
 			(stroke
@@
 		(fp_arc
 			(start 46.63125 -5.499999)
-			(mid 46.777693 -5.853571)
+			(mid 46.777699 -5.853535)
 			(end 47.13125 -5.999999)
 			(stroke
@@
 		(fp_arc
 			(start 47.13125 8.000001)
-			(mid 46.777729 7.853537)
+			(mid 46.777693 7.853543)
 			(end 46.63125 7.500001)
 			(stroke
@@
 		(fp_arc
 			(start 52.880039 -5.999999)
-			(mid 53.233567 -5.853539)
+			(mid 53.233602 -5.853545)
 			(end 53.380039 -5.499999)
 			(stroke
@@
 		(fp_arc
 			(start 53.38125 7.500001)
-			(mid 53.234806 7.853571)
+			(mid 53.2348 7.853536)
 			(end 52.88125 8.000001)
 			(stroke
@@
 		(fp_arc
 			(start 9.03125 8.000001)
-			(mid 8.677729 7.853537)
+			(mid 8.677693 7.853543)
 			(end 8.53125 7.500001)
 			(stroke
@@
 		(fp_arc
 			(start 14.780039 -5.999999)
-			(mid 15.133567 -5.853539)
+			(mid 15.133602 -5.853545)
 			(end 15.280039 -5.499999)
 			(stroke
@@
 		(fp_arc
 			(start 15.28125 7.500001)
-			(mid 15.134806 7.853571)
+			(mid 15.1348 7.853536)
 			(end 14.78125 8.000001)
 			(stroke
@@
 		(fp_arc
 			(start 9.03125 8.000001)
-			(mid 8.677729 7.853537)
+			(mid 8.677693 7.853543)
 			(end 8.53125 7.500001)
 			(stroke
@@
 		(fp_arc
 			(start 14.780039 -5.999999)
-			(mid 15.133567 -5.853539)
+			(mid 15.133602 -5.853545)
 			(end 15.280039 -5.499999)
 			(stroke
@@
 		(fp_arc
 			(start 15.28125 7.500001)
-			(mid 15.134806 7.853571)
+			(mid 15.1348 7.853536)
 			(end 14.78125 8.000001)
 			(stroke
@@
 	)
 	(gr_line
-		(start 371.475 183.35625)
-		(end 362.74375 183.35625)
+		(start 371.475 184.15)
+		(end 362.74375 184.15)
 		(stroke
 			(width 0.05)
@@
 	(gr_line
 		(start 372.26875 126.20625)
-		(end 372.26875 182.5625)
+		(end 372.26875 183.35625)
 		(stroke
 			(width 0.05)
@@
 	(gr_line
 		(start 46.83125 87.3125)
-		(end 46.83125 182.5625)
+		(end 46.83125 183.35625)
 		(stroke
 			(width 0.05)
@@
 	)
 	(gr_arc
-		(start 47.625 183.35625)
-		(mid 47.063734 183.123766)
-		(end 46.83125 182.5625)
+		(start 47.625 184.15)
+		(mid 47.063734 183.917516)
+		(end 46.83125 183.35625)
 		(stroke
 			(width 0.05)
@@
 	)
 	(gr_line
-		(start 47.625 183.35625)
-		(end 362.74375 183.35625)
+		(start 47.625 184.15)
+		(end 362.74375 184.15)
 		(stroke
 			(width 0.05)
@@
 	)
 	(gr_arc
-		(start 372.26875 182.5625)
-		(mid 372.036266 183.123766)
-		(end 371.475 183.35625)
+		(start 372.26875 183.35625)
+		(mid 372.036266 183.917516)
+		(end 371.475 184.15)
 		(stroke
 			(width 0.05)
@@
 	)
 	(segment
-		(start 347.165754 100.359655)
-		(end 345.616465 98.810366)
-		(width 0.2)
-		(layer "F.Cu")
-		(net 1)
-	)
-	(segment
 		(start 345.266465 127.460366)
 		(end 347.866465 130.060366)
@@
 	)
 	(segment
-		(start 347.165754 101.545646)
-		(end 347.165754 100.359655)
+		(start 347.414127 101.794019)
+		(end 347.414127 99.940464)
 		(width 0.2)
 		(layer "F.Cu")
@@
 	)
 	(segment
+		(start 347.414127 99.940464)
+		(end 346.384029 98.910366)
+		(width 0.2)
+		(layer "F.Cu")
+		(net 1)
+	)
+	(segment
 		(start 340.666465 104.410366)
 		(end 344.867936 104.410366)
@@
 	)
 	(via
-		(at 347.165754 101.545646)
+		(at 347.414127 101.794019)
 		(size 0.6)
 		(drill 0.3)
@@
 	)
 	(via
-		(at 345.616465 98.810366)
+		(at 346.384029 98.910366)
 		(size 0.6)
 		(drill 0.3)
@@
 	)
 	(segment
-		(start 346.555215 96.621616)
-		(end 346.116465 97.060366)
+		(start 345.466465 101.460366)
+		(end 347.080474 101.460366)
 		(width 0.2)
 		(layer "B.Cu")
@@
 	)
 	(segment
-		(start 348.100474 102.480366)
-		(end 347.165754 101.545646)
+		(start 346.555215 96.621616)
+		(end 346.116465 97.060366)
 		(width 0.2)
 		(layer "B.Cu")
@@
 	)
 	(segment
-		(start 345.466465 101.460366)
-		(end 347.016465 101.460366)
-		(width 0.2)
-		(layer "B.Cu")
-		(net 1)
-	)
-	(segment
 		(start 348.866465 109.060366)
 		(end 348.866465 110.120366)
@@
 	)
 	(segment
-		(start 348.466465 102.480366)
-		(end 348.100474 102.480366)
-		(width 0.2)
-		(layer "B.Cu")
-		(net 1)
-	)
-	(segment
 		(start 341.310215 89.754116)
 		(end 338.985215 89.754116)
@@
 	)
 	(segment
+		(start 347.080474 101.460366)
+		(end 347.414127 101.794019)
+		(width 0.2)
+		(layer "B.Cu")
+		(net 1)
+	)
+	(segment
 		(start 346.116465 97.292776)
 		(end 346.116465 97.060366)
@@
 	)
 	(segment
+		(start 346.384029 98.910366)
+		(end 346.284029 98.810366)
+		(width 0.2)
+		(layer "B.Cu")
+		(net 1)
+	)
+	(segment
 		(start 347.816465 130.110366)
 		(end 347.866465 130.060366)
@@
 	)
 	(segment
+		(start 347.414127 101.794019)
+		(end 348.100474 102.480366)
+		(width 0.2)
+		(layer "B.Cu")
+		(net 1)
+	)
+	(segment
+		(start 348.100474 102.480366)
+		(end 348.466465 102.480366)
+		(width 0.2)
+		(layer "B.Cu")
+		(net 1)
+	)
+	(segment
 		(start 341.366465 89.810366)
 		(end 341.310215 89.754116)
@@
 	)
 	(segment
-		(start 347.016465 101.460366)
-		(end 347.116465 101.560366)
+		(start 332.616465 88.310366)
+		(end 333.616465 88.310366)
 		(width 0.2)
 		(layer "B.Cu")
@@
 	)
 	(segment
-		(start 332.616465 88.310366)
-		(end 333.616465 88.310366)
+		(start 340.591465 96.310366)
+		(end 340.616465 96.310366)
 		(width 0.2)
 		(layer "B.Cu")
@@
 	)
 	(segment
-		(start 340.591465 96.310366)
-		(end 340.616465 96.310366)
+		(start 346.284029 98.810366)
+		(end 344.598875 98.810366)
 		(width 0.2)
 		(layer "B.Cu")
@@
 	)
 	(segment
-		(start 345.616465 98.810366)
-		(end 344.598875 98.810366)
-		(width 0.2)
-		(layer "B.Cu")
-		(net 1)
-	)
-	(segment
 		(start 342.028965 109.010366)
 		(end 342.028965 107.122866)
@@
 	)
 	(segment
-		(start 350.900779 115.960366)
-		(end 352.466465 114.39468)
+		(start 352.466465 109.824581)
+		(end 350.616465 107.974581)
+		(width 0.2)
+		(layer "F.Cu")
+		(net 94)
+	)
+	(segment
+		(start 343.482585 99.310366)
+		(end 342.374525 98.202306)
+		(width 0.2)
+		(layer "F.Cu")
+		(net 94)
+	)
+	(segment
+		(start 350.566465 119.560366)
+		(end 350.900779 119.226052)
 		(width 0.2)
 		(layer "F.Cu")
@@
 	(segment
 		(start 350.616465 107.974581)
-		(end 350.616465 106.444246)
+		(end 350.616465 103.760215)
 		(width 0.2)
 		(layer "F.Cu")
@@
 	)
 	(segment
-		(start 350.616465 106.444246)
-		(end 342.374525 98.202306)
+		(start 352.466465 114.39468)
+		(end 352.466465 109.824581)
 		(width 0.2)
 		(layer "F.Cu")
@@
 	)
 	(segment
-		(start 350.900779 119.226052)
-		(end 350.900779 115.960366)
+		(start 350.616465 103.760215)
+		(end 348.673216 103.760215)
 		(width 0.2)
 		(layer "F.Cu")
@@
 	)
 	(segment
-		(start 352.466465 109.824581)
-		(end 350.616465 107.974581)
+		(start 346.076922 99.310366)
+		(end 343.482585 99.310366)
 		(width 0.2)
 		(layer "F.Cu")
@@
 	)
 	(segment
-		(start 350.566465 119.560366)
-		(end 350.900779 119.226052)
+		(start 348.673216 103.760215)
+		(end 346.86875 101.955749)
 		(width 0.2)
 		(layer "F.Cu")
@@
 	)
 	(segment
-		(start 352.466465 114.39468)
-		(end 352.466465 109.824581)
+		(start 346.86875 100.102194)
+		(end 346.076922 99.310366)
+		(width 0.2)
+		(layer "F.Cu")
+		(net 94)
+	)
+	(segment
+		(start 350.900779 119.226052)
+		(end 350.900779 115.960366)
+		(width 0.2)
+		(layer "F.Cu")
+		(net 94)
+	)
+	(segment
+		(start 346.86875 101.955749)
+		(end 346.86875 100.102194)
+		(width 0.2)
+		(layer "F.Cu")
+		(net 94)
+	)
+	(segment
+		(start 350.900779 115.960366)
+		(end 352.466465 114.39468)
 		(width 0.2)
 		(layer "F.Cu")

Commit message: updated file structure ish
Parts:
- added G***: LOGO, 8.0:front, F.Cu at (209.6, 134.9)
- added G***: LOGO, 8.0:name, B.Cu at (352.7, 155.3)
- added G***: LOGO, 8.0:QMK, B.Cu at (362.7, 153.2)
- moved C3 2.49 mm to (354.5, 109.8)
- moved C4 2.05 mm to (354.5, 112.4)
- moved C12 0.34 mm to (346.2, 115.5)
Routing:
- net GND: track 156.7 -> 161.8 mm
- net Net-(U3-VREG_VOUT): track 51.0 -> 54.8 mm
Other:
- outline, holes or cut-outs redrawn

Commit message: reordered, x3, hopefully final production
Parts:
- R1, R2, R3, R4, R5, R6, R7, R8: footprint Resistor_SMD:R_01005_0402Metric -> Resistor_SMD:R_0402_1005Metric
- moved R8 0.47 mm to (339.4, 132.6)
- moved R7 0.38 mm to (342.8, 104.8)
- moved R1 0.32 mm to (340.8, 97.3)
- moved SW1 0.17 mm to (350.8, 131.9)
- moved R2 0.13 mm to (346.0, 97.1)
Routing:
- net GND: track 161.8 -> 161.0 mm
- net Net-(U3-RUN): track 70.6 -> 71.2 mm
